Commit message: and look at

File: src/dream_ros2_bridge/urdf/xarm6.urdf (robot description, URDF)
Before this commit: robot UF_ROBOT, 9 links, 8 joints
Links:
- removed link world
- added link arm_base
Joints:
- removed joint world_joint
- added joint arm_base_joint: type fixed, parent arm_base, child link_base, origin xyz=0 0 0 rpy=0 0 0
