Commit message: update urdf file

File: src/dream_ros2_bridge/urdf/rangerminiv3_with_xarm6_tmp.urdf (robot description, URDF)
Before this commit: robot ranger_mini_v3, 18 links, 17 joints
Links:
- link base_link: geometry collision box size=0.738 0.5 0.24; visual mesh filename=/home/yanzj/workspace/DREAM/src/dream_ros2_bridge/meshes/ra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
- link fl_steering_wheel_link: geometry collision cylinder length=0.001 radius=0.001; visual mesh filename=/home/yanzj/workspace/DREAM/src/dream_ros2_bridge/meshes/ra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
- link fr_steering_wheel_link: geometry collision cylinder length=0.001 radius=0.001; visual mesh filename=/home/yanzj/workspace/DREAM/src/dream_ros2_bridge/meshes/ra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
- link link1: geometry collision mesh filename=/home/yanzj/workspace/DREAM/src/dream_ros2_bridge/meshes/li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; visual mesh filename=/home/yanzj/workspace/DREAM/src/dream_ros2_bridge/meshes/li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
- link link2: geometry collision mesh filename=/home/yanzj/workspace/DREAM/src/dream_ros2_bridge/meshes/li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; visual mesh filename=/home/yanzj/workspace/DREAM/src/dream_ros2_bridge/meshes/li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
- link link3: geometry collision mesh filename=/home/yanzj/workspace/DREAM/src/dream_ros2_bridge/meshes/li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; visual mesh filename=/home/yanzj/workspace/DREAM/src/dream_ros2_bridge/meshes/li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
- link link4: geometry collision mesh filename=/home/yanzj/workspace/DREAM/src/dream_ros2_bridge/meshes/li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; visual mesh filename=/home/yanzj/workspace/DREAM/src/dream_ros2_bridge/meshes/li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
- link link5: geometry collision mesh filename=/home/yanzj/workspace/DREAM/src/dream_ros2_bridge/meshes/li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; visual mesh filename=/home/yanzj/workspace/DREAM/src/dream_ros2_bridge/meshes/li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
- link link6: geometry collision mesh filename=/home/yanzj/workspace/DREAM/src/dream_ros2_bridge/meshes/en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; visual mesh filename=/home/yanzj/workspace/DREAM/src/dream_ros2_bridge/meshes/li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
- link link_base: geometry collision mesh filename=/home/yanzj/workspace/DREAM/src/dream_ros2_bridge/meshes/li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; visual mesh filename=/home/yanzj/workspace/DREAM/src/dream_ros2_bridge/meshes/li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
- link rl_steering_wheel_link: geometry collision cylinder length=0.001 radius=0.001; visual mesh filename=/home/yanzj/workspace/DREAM/src/dream_ros2_bridge/meshes/ra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
- link rr_steering_wheel_link: geometry collision cylinder length=0.001 radius=0.001; visual mesh filename=/home/yanzj/workspace/DREAM/src/dream_ros2_bridge/meshes/ra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

Commit message: udpate

File: src/dream_ros2_bridge/urdf/rangerminiv3_with_xarm6_tmp.urdf (robot description, URDF)
Before this commit: robot ranger_mini_v3, 18 links, 17 joints
Links:
- link base_link: geometry collision box size=0.738 0.5 0.24; visual mesh filename=src/dream_ros2_bridge/meshes/ranger_mini3.dae
- link fl_steering_wheel_link: geometry collision cylinder length=0.001 radius=0.001; visual mesh filename=src/dream_ros2_bridge/meshes/ranger_mini_v3_wheel.dae
- link fr_steering_wheel_link: geometry collision cylinder length=0.001 radius=0.001; visual mesh filename=src/dream_ros2_bridge/meshes/ranger_mini_v3_wheel_right.dae
- link link1: geometry collision mesh filename=src/dream_ros2_bridge/meshes/link1.stl; visual mesh filename=src/dream_ros2_bridge/meshes/link1.stl
- link link2: geometry collision mesh filename=src/dream_ros2_bridge/meshes/link2.stl; visual mesh filename=src/dream_ros2_bridge/meshes/link2.stl
- link link3: geometry collision mesh filename=src/dream_ros2_bridge/meshes/link3.stl; visual mesh filename=src/dream_ros2_bridge/meshes/link3.stl
- link link4: geometry collision mesh filename=src/dream_ros2_bridge/meshes/link4.stl; visual mesh filename=src/dream_ros2_bridge/meshes/link4.stl
- link link5: geometry collision mesh filename=src/dream_ros2_bridge/meshes/link5.stl; visual mesh filename=src/dream_ros2_bridge/meshes/link5.stl
- link link6: geometry collision mesh filename=src/dream_ros2_bridge/meshes/end_tool.stl; visual mesh filename=src/dream_ros2_bridge/meshes/link6.stl
- link link_base: geometry collision mesh filename=src/dream_ros2_bridge/meshes/link_base.stl; visual mesh filename=src/dream_ros2_bridge/meshes/link_base.stl
- link rl_steering_wheel_link: geometry collision cylinder length=0.001 radius=0.001; visual mesh filename=src/dream_ros2_bridge/meshes/ranger_mini_v3_wheel.dae
- link rr_steering_wheel_link: geometry collision cylinder length=0.001 radius=0.001; visual mesh filename=src/dream_ros2_bridge/meshes/ranger_mini_v3_wheel_right.dae
